Commit message: feat: modified inertial values

File: urdf/base.xacro (robot description, xacro)
@@ -17,6 +17,6 @@
       </collision>
       <inertial>
-        <mass value="1.0" />
-        <inertia ixx="0.015" ixy="0" ixz="0" iyy="0.0375" iyz="0.0" izz="0.0375" />
+        <mass value="0.5" />
+        <inertia ixx="0.015" ixy="0" ixz="0" iyy="0.0375" iyz="0.0" izz="0.0275" />
       </inertial>
     </link>

File: urdf/lidar.xacro (robot description, xacro)
@@ -17,6 +17,6 @@
       </collision>
       <inertial>
-        <mass value="1.0" />
-        <inertia ixx="0.015" ixy="0" ixz="0" iyy="0.0375" iyz="0.0" izz="0.0375" />
+        <mass value="0.01" />
+        <inertia ixx="0.015" ixy="0" ixz="0" iyy="0.0375" iyz="0.0" izz="0.0275" />
       </inertial>
     </link>

File: urdf/motor.xacro (robot description, xacro)
@@ -17,6 +17,6 @@
       </collision>
       <inertial>
-        <mass value="1.0" />
-        <inertia ixx="0.015" ixy="0" ixz="0" iyy="0.0375" iyz="0.0" izz="0.0375" />
+        <mass value="0.2" />
+        <inertia ixx="0.015" ixy="0" ixz="0" iyy="0.0375" iyz="0.0" izz="0.0275" />
       </inertial>
     </link>

File: urdf/pillar.xacro (robot description, xacro)
@@ -17,6 +17,6 @@
       </collision>
       <inertial>
-        <mass value="1.0" />
-        <inertia ixx="0.015" ixy="0" ixz="0" iyy="0.0375" iyz="0.0" izz="0.0375" />
+        <mass value="0.1" />
+        <inertia ixx="0.015" ixy="0" ixz="0" iyy="0.0375" iyz="0.0" izz="0.0275" />
       </inertial>
     </link>

File: urdf/robot.xacro (robot description, xacro)
@@ -57,5 +57,5 @@
         <wheel_diameter>0.035</wheel_diameter>
         <wheel_diameter>0.035</wheel_diameter>
-        <max_wheel_torque>200</max_wheel_torque>
+        <max_wheel_torque>50</max_wheel_torque>
         <max_wheel_acceleration>10.0</max_wheel_acceleration>
         <odometry_frame>odom</odometry_frame>

File: urdf/wheel.xacro (robot description, xacro)
@@ -17,6 +17,6 @@
       </collision>
       <inertial>
-        <mass value="1.0" />
-        <inertia ixx="0.015" ixy="0" ixz="0" iyy="0.0375" iyz="0.0" izz="0.0375" />
+        <mass value="0.1" />
+        <inertia ixx="0.015" ixy="0" ixz="0" iyy="0.0375" iyz="0.0" izz="0.0275" />
       </inertial>
     </link>
