Commit message: Added gazebo plugin for lidar

File: urdf/lidar.xacro (robot description, xacro)
@@ -26,4 +26,38 @@
       <child link="${child}" />
     </joint>
+    <gazebo reference="${child}">
+      <sensor name="lidar" type="ray">
+        <always_on>true</always_on>
+        <visualize>true</visualize>
+        <update_rate>5</update_rate>
+        <ray>
+          <scan>
+            <horizontal>
+              <samples>360</samples>
+              <resolution>1.000000</resolution>
+              <min_angle>0.000000</min_angle>
+              <max_angle>6.280000</max_angle>
+            </horizontal>
+          </scan>
+          <range>
+            <min>0.120000</min>
+            <max>3.5</max>
+            <resolution>0.015000</resolution>
+          </range>
+          <noise>
+            <type>gaussian</type>
+            <mean>0.0</mean>
+            <stddev>0.01</stddev>
+          </noise>
+        </ray>
+        <plugin name="scan" filename="libgazebo_ros_ray_sensor.so">
+          <ros>
+            <remapping>~/out:=scan</remapping>
+          </ros>
+          <output_type>sensor_msgs/LaserScan</output_type>
+          <frame_name>${child}</frame_name>
+        </plugin>
+      </sensor>
+    </gazebo>
   </xacro:macro>
 </robot>

File: urdf/motor.xacro (robot description, xacro)
@@ -17,5 +17,5 @@
       </collision>
       <inertial>
-        <mass value="0.2" />
+        <mass value="1.5" />
         <inertia ixx="0.015" ixy="0" ixz="0" iyy="0.0375" iyz="0.0" izz="0.0275" />
       </inertial>

File: urdf/robot.xacro (robot description, xacro)
@@ -33,8 +33,8 @@
       <plugin name="object_controller" filename="libgazebo_ros_planar_move.so">
         <ros>
-          <argument>odom:=odom/unfiltered</argument>
+          <argument>odom:=odom</argument>
         </ros>
         <command_topic>cmd_vel</command_topic>
-        <odometry_topic>odom/unfiltered</odometry_topic>
+        <odometry_topic>odom</odometry_topic>
         <odometry_frame>odom</odometry_frame>
         <odometry_rate>20.0</odometry_rate>
